Commit message: added gazebo controller, created a launch file launch_sim and created a gazebo world

File: description/robot.urdf.xacro (robot description, xacro)
@@ -2,3 +2,4 @@
 <robot xmlns:xacro="http://www.ros.org/wiki/xacro"  name="robot">
     <xacro:include filename="robot_core.xacro"/>
+    <xacro:include filename="gazebo_control.xacro" />
 </robot>

File: description/robot_core.xacro (robot description, xacro)
@@ -43,6 +43,11 @@
         </xacro:inertial_box>
     </link>
+<gazebo reference='chassis'>
+    <material>
+        Gazebo/White
+    </material>
+</gazebo>
 <!-- Left Wheel Link-->
-    <joint name="left_wheel_link" type="continuous">
+    <joint name="left_wheel_joint" type="continuous">
         <parent link="base_link"/>
         <child link="left_wheel"/>
@@ -69,6 +74,11 @@
 </xacro:inertial_cylinder>
     </link>
+    <gazebo reference='left_wheel'>
+        <material>
+            Gazebo/Blue
+        </material>
+    </gazebo>
     <!-- Right Wheel Link-->
-    <joint name="right_wheel_link" type="continuous">
+    <joint name="right_wheel_joint" type="continuous">
         <parent link="base_link"/>
         <child link="right_wheel"/>
@@ -95,4 +105,9 @@
 </xacro:inertial_cylinder>
     </link>
+    <gazebo reference='right_wheel'>
+        <material>
+            Gazebo/Blue
+        </material>
+    </gazebo>
 <!-- Caster Wheel Link-->
 <joint name="caster_wheel_joint" type="fixed">
@@ -120,3 +135,11 @@
 </xacro:inertial_sphere>
 </link>
+<gazebo reference='caster_wheel'>
+    <material>
+        Gazebo/Black
+    </material>
+    <!-- friction coef for the caster wheel so they bounce around -->
+    <mu1 value='0.001'/>
+    <mu2 value='001'/>
+</gazebo>
 </robot>
